File: TheGitboard2.0.kicad_pcb (KiCad board)
At the start: 2 copper layers, 78.3 x 70.1 mm, 9 parts, among them SW1 SW_Push, SW2 SW_Push, SW3 SW_Push, SW4 SW_Push, SW5 SW_Push, SW6 SW_Push, SW7 SW_Push, SW8 SW_Push, U1 MOUDLE-SEEEDUINO-XIAO

Commit message: Autosave
Routing:
- net Net-(SW1-Pad2): track 38.1 -> 57.2 mm
Changed lines of the file:
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@@
+	)
+	(segment
+		(start 124.445 105.935)
+		(end 143.495 105.935)
+		(width 0.2)
+		(layer "F.Cu")
+		(net "Net-(SW1-Pad2)")
 	)
 	(segment

Commit message: Autosave
Routing:
- net Net-(U1-PA7_A8_D8_SCK): track 57.2 -> 77.2 mm
Changed lines of the file:
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@@
+	)
+	(segment
+		(start 162.545 103.67403)
+		(end 162.545 105.935)
+		(width 0.2)
+		(layer "F.Cu")
+		(net "Net-(U1-PA7_A8_D8_SCK)")
+	)
+	(segment
+		(start 149.975 91.10403)
+		(end 162.545 103.67403)
+		(width 0.2)
+		(layer "F.Cu")
+		(net "Net-(U1-PA7_A8_D8_SCK)")
 	)
 	(segment

Commit message: Autosave
Routing:
- net Net-(U1-PA5_A9_D9_MISO): track 0.00 -> 58.3 mm
Changed lines of the file:
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@@
+	)
+	(segment
+		(start 132.15597 88.56403)
+		(end 149.975 88.56403)
+		(width 0.2)
+		(layer "F.Cu")
+		(net "Net-(U1-PA5_A9_D9_MISO)")
+	)
+	(segment
+		(start 130.795 89.925)
+		(end 132.15597 88.56403)
+		(width 0.2)
+		(layer "F.Cu")
+		(net "Net-(U1-PA5_A9_D9_MISO)")
+	)
+	(segment
+		(start 130.795 103.395)
+		(end 130.795 89.925)
+		(width 0.2)
+		(layer "F.Cu")
+		(net "Net-(U1-PA5_A9_D9_MISO)")
+	)
+	(segment
+		(start 154.06403 88.56403)
+		(end 168.895 103.395)
+		(width 0.2)
+		(layer "F.Cu")
+		(net "Net-(U1-PA5_A9_D9_MISO)")
+	)
+	(segment
+		(start 149.975 88.56403)
+		(end 154.06403 88.56403)
+		(width 0.2)
+		(layer "F.Cu")
+		(net "Net-(U1-PA5_A9_D9_MISO)")
 	)
 	(segment

Commit message: Autosave
Routing:
- net Net-(U1-PA6_A10_D10_MOSI): track 0.00 -> 103.7 mm
Changed lines of the file:
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@@
+	)
+	(segment
+		(start 134.130284 86.02403)
+		(end 121.975 98.179314)
+		(width 0.2)
+		(layer "F.Cu")
+		(net "Net-(U1-PA6_A10_D10_MOSI)")
+	)
+	(segment
+		(start 127.366598 129.96)
+		(end 141.487056 129.96)
+		(width 0.2)
+		(layer "F.Cu")
+		(net "Net-(U1-PA6_A10_D10_MOSI)")
+	)
+	(segment
+		(start 145.29 124.3)
+		(end 143.435 122.445)
+		(width 0.2)
+		(layer "F.Cu")
+		(net "Net-(U1-PA6_A10_D10_MOSI)")
+	)
+	(segment
+		(start 121.975 98.179314)
+		(end 121.975 124.568402)
+		(width 0.2)
+		(layer "F.Cu")
+		(net "Net-(U1-PA6_A10_D10_MOSI)")
+	)
+	(segment
+		(start 141.487056 129.96)
+		(end 145.29 126.157056)
+		(width 0.2)
+		(layer "F.Cu")
+		(net "Net-(U1-PA6_A10_D10_MOSI)")
+	)
+	(segment
+		(start 143.435 122.445)
+		(end 130.795 122.445)
+		(width 0.2)
+		(layer "F.Cu")
+		(net "Net-(U1-PA6_A10_D10_MOSI)")
+	)
+	(segment
+		(start 145.29 126.157056)
+		(end 145.29 124.3)
+		(width 0.2)
+		(layer "F.Cu")
+		(net "Net-(U1-PA6_A10_D10_MOSI)")
+	)
+	(segment
+		(start 149.975 86.02403)
+		(end 134.130284 86.02403)
+		(width 0.2)
+		(layer "F.Cu")
+		(net "Net-(U1-PA6_A10_D10_MOSI)")
+	)
+	(segment
+		(start 121.975 124.568402)
+		(end 127.366598 129.96)
+		(width 0.2)
+		(layer "F.Cu")
+		(net "Net-(U1-PA6_A10_D10_MOSI)")
 	)
 	(segment

Commit message: Autosave
Routing:
- net Net-(U1-PA6_A10_D10_MOSI): track 103.7 -> 169.2 mm
Changed lines of the file:
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@@
+	)
+	(segment
+		(start 168.965 101.995)
+		(end 182.307944 101.995)
+		(width 0.2)
+		(layer "F.Cu")
+		(net "Net-(U1-PA6_A10_D10_MOSI)")
 	)
 	(segment
 		(start 134.130284 86.02403)
 		(end 121.975 98.179314)
+		(width 0.2)
+		(layer "F.Cu")
+		(net "Net-(U1-PA6_A10_D10_MOSI)")
+	)
+	(segment
+		(start 152.99403 86.02403)
+		(end 168.965 101.995)
 		(width 0.2)
 		(layer "F.Cu")
@@
 		(width 0.2)
 		(layer "F.Cu")
+		(net "Net-(U1-PA6_A10_D10_MOSI)")
+	)
+	(segment
+		(start 149.975 86.02403)
+		(end 152.99403 86.02403)
+		(width 0.2)
+		(layer "F.Cu")
+		(net "Net-(U1-PA6_A10_D10_MOSI)")
+	)
+	(segment
+		(start 182.995 102.682056)
+		(end 182.995 108.345)
+		(width 0.2)
+		(layer "F.Cu")
+		(net "Net-(U1-PA6_A10_D10_MOSI)")
+	)
+	(segment
+		(start 182.995 108.345)
+		(end 168.895 122.445)
+		(width 0.2)
+		(layer "F.Cu")
+		(net "Net-(U1-PA6_A10_D10_MOSI)")
+	)
+	(segment
+		(start 182.307944 101.995)
+		(end 182.995 102.682056)
+		(width 0.2)
+		(layer "F.Cu")

Commit message: Autosave
Routing:
- net Net-(U1-PA6_A10_D10_MOSI): track 169.2 -> 0.00 mm
- net Net-(U1-PA5_A9_D9_MISO): track 58.3 -> 0.00 mm
- net Net-(SW1-Pad2): track 57.2 -> 0.00 mm
Changed lines of the file:
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@@
-	)
-	(segment
-		(start 132.15597 88.56403)
-		(end 149.975 88.56403)
-		(width 0.2)
-		(layer "F.Cu")
-		(net "Net-(U1-PA5_A9_D9_MISO)")
-	)
-	(segment
-		(start 130.795 89.925)
-		(end 132.15597 88.56403)
-		(width 0.2)
-		(layer "F.Cu")
-		(net "Net-(U1-PA5_A9_D9_MISO)")
-	)
-	(segment
-		(start 130.795 103.395)
-		(end 130.795 89.925)
-		(width 0.2)
-		(layer "F.Cu")
-		(net "Net-(U1-PA5_A9_D9_MISO)")
-	)
-	(segment
-		(start 154.06403 88.56403)
-		(end 168.895 103.395)
-		(width 0.2)
-		(layer "F.Cu")
-		(net "Net-(U1-PA5_A9_D9_MISO)")
-	)
-	(segment
-		(start 149.975 88.56403)
-		(end 154.06403 88.56403)
-		(width 0.2)
-		(layer "F.Cu")
-		(net "Net-(U1-PA5_A9_D9_MISO)")
 	)
 	(segment
@@
 		(net "Net-(U1-PA7_A8_D8_SCK)")
 	)
-	(segment
-		(start 168.965 101.995)
-		(end 182.307944 101.995)
-		(width 0.2)
-		(layer "F.Cu")
-		(net "Net-(U1-PA6_A10_D10_MOSI)")
-	)
-	(segment
-		(start 134.130284 86.02403)
-		(end 121.975 98.179314)
-		(width 0.2)
-		(layer "F.Cu")
-		(net "Net-(U1-PA6_A10_D10_MOSI)")
-	)
-	(segment
-		(start 152.99403 86.02403)
-		(end 168.965 101.995)
-		(width 0.2)
-		(layer "F.Cu")
-		(net "Net-(U1-PA6_A10_D10_MOSI)")
-	)
-	(segment
-		(start 127.366598 129.96)
-		(end 141.487056 129.96)
-		(width 0.2)
-		(layer "F.Cu")
-		(net "Net-(U1-PA6_A10_D10_MOSI)")
-	)
-	(segment
-		(start 145.29 124.3)
-		(end 143.435 122.445)
-		(width 0.2)
-		(layer "F.Cu")
-		(net "Net-(U1-PA6_A10_D10_MOSI)")
-	)
-	(segment
-		(start 149.975 86.02403)
-		(end 152.99403 86.02403)
-		(width 0.2)
-		(layer "F.Cu")
-		(net "Net-(U1-PA6_A10_D10_MOSI)")
-	)
-	(segment
-		(start 182.995 102.682056)
-		(end 182.995 108.345)
-		(width 0.2)
-		(layer "F.Cu")
-		(net "Net-(U1-PA6_A10_D10_MOSI)")
-	)
-	(segment
-		(start 182.995 108.345)
-		(end 168.895 122.445)
-		(width 0.2)
-		(layer "F.Cu")
-		(net "Net-(U1-PA6_A10_D10_MOSI)")
-	)
-	(segment
-		(start 182.307944 101.995)
-		(end 182.995 102.682056)
-		(width 0.2)
-		(layer "F.Cu")
-		(net "Net-(U1-PA6_A10_D10_MOSI)")
-	)
-	(segment
-		(start 121.975 98.179314)
-		(end 121.975 124.568402)
-		(width 0.2)
-		(layer "F.Cu")
-		(net "Net-(U1-PA6_A10_D10_MOSI)")
-	)
-	(segment
-		(start 141.487056 129.96)
-		(end 145.29 126.157056)
-		(width 0.2)
-		(layer "F.Cu")
-		(net "Net-(U1-PA6_A10_D10_MOSI)")
-	)
-	(segment
-		(start 143.435 122.445)
-		(end 130.795 122.445)
-		(width 0.2)
-		(layer "F.Cu")
-		(net "Net-(U1-PA6_A10_D10_MOSI)")
-	)
-	(segment
-		(start 145.29 126.157056)
-		(end 145.29 124.3)
-		(width 0.2)
-		(layer "F.Cu")
-		(net "Net-(U1-PA6_A10_D10_MOSI)")
-	)
-	(segment
-		(start 149.975 86.02403)
-		(end 134.130284 86.02403)
-		(width 0.2)
-		(layer "F.Cu")
-		(net "Net-(U1-PA6_A10_D10_MOSI)")
-	)
-	(segment
-		(start 121.975 124.568402)
-		(end 127.366598 129.96)
-		(width 0.2)
-		(layer "F.Cu")
-		(net "Net-(U1-PA6_A10_D10_MOSI)")
-	)
-	(segment
-		(start 124.445 105.935)
-		(end 143.495 105.935)
-		(width 0.2)
-		(layer "F.Cu")
-		(net "Net-(SW1-Pad2)")
-	)
-	(segment
-		(start 124.445 124.985)
-		(end 143.495 124.985)
-		(width 0.2)
-		(layer "F.Cu")
-		(net "Net-(SW1-Pad2)")
-	)
-	(segment
-		(start 124.445 105.935)
-		(end 124.445 124.985)
-		(width 0.2)
-		(layer "F.Cu")
-		(net "Net-(SW1-Pad2)")
-	)
 	(embedded_fonts no)

Commit message: Autosave
Routing:
- net Net-(U1-PA7_A8_D8_SCK): track 77.2 -> 0.00 mm
Changed lines of the file:
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@@
 		(layer "Edge.Cuts")
-	)
-	(segment
-		(start 162.545 105.935)
-		(end 162.545 124.985)
-		(width 0.2)
-		(layer "F.Cu")
-		(net "Net-(U1-PA7_A8_D8_SCK)")
-	)
-	(segment
-		(start 181.595 124.985)
-		(end 162.545 124.985)
-		(width 0.2)
-		(layer "F.Cu")
-		(net "Net-(U1-PA7_A8_D8_SCK)")
-	)
-	(segment
-		(start 162.545 105.935)
-		(end 181.595 105.935)
-		(width 0.2)
-		(layer "F.Cu")
-		(net "Net-(U1-PA7_A8_D8_SCK)")
-	)
-	(segment
-		(start 162.545 103.67403)
-		(end 162.545 105.935)
-		(width 0.2)
-		(layer "F.Cu")
-		(net "Net-(U1-PA7_A8_D8_SCK)")
-	)
-	(segment
-		(start 149.975 91.10403)
-		(end 162.545 103.67403)
-		(width 0.2)
-		(layer "F.Cu")
-		(net "Net-(U1-PA7_A8_D8_SCK)")
 	)
 	(embedded_fonts no)

Commit message: Autosave
Routing:
- net Net-(U1-PA7_A8_D8_SCK): track 0.00 -> 57.2 mm
Changed lines of the file:
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@@
 		(layer "Edge.Cuts")
+	)
+	(segment
+		(start 181.595 105.935)
+		(end 162.545 105.935)
+		(width 0.2)
+		(layer "F.Cu")
+		(net "Net-(U1-PA7_A8_D8_SCK)")
+	)
+	(segment
+		(start 181.595 124.985)
+		(end 162.545 124.985)
+		(width 0.2)
+		(layer "F.Cu")
+		(net "Net-(U1-PA7_A8_D8_SCK)")
+	)
+	(segment
+		(start 162.545 124.985)
+		(end 162.545 105.935)
+		(width 0.2)
+		(layer "F.Cu")
+		(net "Net-(U1-PA7_A8_D8_SCK)")
 	)
 	(embedded_fonts no)
