File: TheGitboard2.0.kicad_pcb (KiCad board)
At the start: 2 copper layers, 78.3 x 70.1 mm, 9 parts, among them SW1 SW_Push, SW2 SW_Push, SW3 SW_Push, SW4 SW_Push, SW5 SW_Push, SW6 SW_Push, SW7 SW_Push, SW8 SW_Push, U1 MOUDLE-SEEEDUINO-XIAO

Commit message: Autosave
Routing:
- net Net-(U1-3V3): track 89.7 -> 191.3 mm
Changed lines of the file:
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@@
+	)
+	(segment
+		(start 186.545 123.024899)
+		(end 187.365101 123.845)
+		(width 0.2)
+		(layer "F.Cu")
+		(net "Net-(U1-3V3)")
+	)
+	(segment
+		(start 167.495 119.607944)
+		(end 167.495 123.024899)
+		(width 0.2)
+		(layer "F.Cu")
+		(net "Net-(U1-3V3)")
+	)
+	(segment
+		(start 169.474899 123.845)
+		(end 170.295 123.024899)
+		(width 0.2)
+		(layer "F.Cu")
+		(net "Net-(U1-3V3)")
 	)
 	(segment
 		(start 193.14 130.16)
-		(end 193.14 108.59)
+		(end 193.14 119.229899)
+		(width 0.2)
+		(layer "F.Cu")
+		(net "Net-(U1-3V3)")
+	)
+	(segment
+		(start 180.822056 107.275)
+		(end 179.827944 107.275)
+		(width 0.2)
+		(layer "F.Cu")
+		(net "Net-(U1-3V3)")
+	)
+	(segment
+		(start 182.012968 107.977944)
+		(end 181.525 107.977944)
+		(width 0.2)
+		(layer "F.Cu")
+		(net "Net-(U1-3V3)")
+	)
+	(segment
+		(start 181.525 107.977944)
+		(end 180.822056 107.275)
 		(width 0.2)
 		(layer "F.Cu")
@@
 	)
 	(segment
+		(start 188.524899 123.845)
+		(end 193.14 119.229899)
+		(width 0.2)
+		(layer "F.Cu")
+		(net "Net-(U1-3V3)")
+	)
+	(segment
+		(start 168.315101 123.845)
+		(end 169.474899 123.845)
+		(width 0.2)
+		(layer "F.Cu")
+		(net "Net-(U1-3V3)")
+	)
+	(segment
+		(start 193.14 119.229899)
+		(end 193.14 108.59)
+		(width 0.2)
+		(layer "F.Cu")
+		(net "Net-(U1-3V3)")
+	)
+	(segment
 		(start 165.666598 130.16)
 		(end 193.14 130.16)
+		(width 0.2)
+		(layer "F.Cu")
+		(net "Net-(U1-3V3)")
+	)
+	(segment
+		(start 185.745 104.245912)
+		(end 182.012968 107.977944)
+		(width 0.2)
+		(layer "F.Cu")
+		(net "Net-(U1-3V3)")
+	)
+	(segment
+		(start 182.694088 101.195)
+		(end 185.745 104.245912)
+		(width 0.2)
+		(layer "F.Cu")
+		(net "Net-(U1-3V3)")
+	)
+	(segment
+		(start 170.295 123.024899)
+		(end 186.545 123.024899)
 		(width 0.2)
 		(layer "F.Cu")
@@
 		(width 0.2)
 		(layer "F.Cu")
+		(net "Net-(U1-3V3)")
+	)
+	(segment
+		(start 167.68597 101.195)
+		(end 182.694088 101.195)
+		(width 0.2)
+		(layer "F.Cu")
+		(net "Net-(U1-3V3)")
+	)
+	(segment
+		(start 179.827944 107.275)
+		(end 167.495 119.607944)
+		(width 0.2)
+		(layer "F.Cu")
+		(net "Net-(U1-3V3)")
+	)
+	(segment
+		(start 167.495 123.024899)
+		(end 168.315101 123.845)
+		(width 0.2)
+		(layer "F.Cu")
+		(net "Net-(U1-3V3)")
+	)
+	(segment
+		(start 149.975 83.48403)
+		(end 167.68597 101.195)
+		(width 0.2)
+		(layer "F.Cu")
+		(net "Net-(U1-3V3)")
+	)
+	(segment
+		(start 187.365101 123.845)
+		(end 188.524899 123.845)
+		(width 0.2)
+		(layer "F.Cu")

Commit message: Autosave
Routing:
- net Net-(U1-3V3): track 191.3 -> 0.00 mm
- net Net-(U1-GND): track 169.2 -> 0.00 mm
- net Net-(U1-PA6_A10_D10_MOSI): track 130.3 -> 0.00 mm
- net Net-(SW1-Pad2): track 57.2 -> 0.00 mm
- net Net-(U1-PA5_A9_D9_MISO): track 50.4 -> 0.00 mm
- net Net-(U1-PA7_A8_D8_SCK): track 77.2 -> 57.2 mm

Commit message: Autosave
Routing:
- net Net-(U1-PA7_A8_D8_SCK): track 57.2 -> 77.2 mm
Changed lines of the file:
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@@
+	)
+	(segment
+		(start 162.545 105.935)
+		(end 162.545 103.67403)
+		(width 0.2)
+		(layer "F.Cu")
+		(net "Net-(U1-PA7_A8_D8_SCK)")
+	)
+	(segment
+		(start 162.545 103.67403)
+		(end 149.975 91.10403)
+		(width 0.2)
+		(layer "F.Cu")
+		(net "Net-(U1-PA7_A8_D8_SCK)")
 	)
 	(segment

Commit message: Autosave
Routing:
- net Net-(U1-3V3): track 0.00 -> 89.7 mm
Changed lines of the file:
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@@
 		(net "Net-(U1-PA7_A8_D8_SCK)")
+	)
+	(segment
+		(start 193.14 130.16)
+		(end 193.14 108.59)
+		(width 0.2)
+		(layer "F.Cu")
+		(net "Net-(U1-3V3)")
+	)
+	(segment
+		(start 149.845 103.395)
+		(end 149.845 114.338402)
+		(width 0.2)
+		(layer "F.Cu")
+		(net "Net-(U1-3V3)")
+	)
+	(segment
+		(start 165.666598 130.16)
+		(end 193.14 130.16)
+		(width 0.2)
+		(layer "F.Cu")
+		(net "Net-(U1-3V3)")
+	)
+	(segment
+		(start 149.845 114.338402)
+		(end 165.666598 130.16)
+		(width 0.2)
+		(layer "F.Cu")
+		(net "Net-(U1-3V3)")
+	)
+	(segment
+		(start 193.14 108.59)
+		(end 187.945 103.395)
+		(width 0.2)
+		(layer "F.Cu")
+		(net "Net-(U1-3V3)")
 	)
 	(embedded_fonts no)

Commit message: Autosave
Routing:
- net Net-(U1-GND): track 0.00 -> 100.2 mm
Changed lines of the file:
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@@
 		(net "Net-(U1-3V3)")
+	)
+	(segment
+		(start 188.745 101.995)
+		(end 193.54 106.79)
+		(width 0.2)
+		(layer "F.Cu")
+		(net "Net-(U1-GND)")
+	)
+	(segment
+		(start 186.545 106.255)
+		(end 186.545 102.815101)
+		(width 0.2)
+		(layer "F.Cu")
+		(net "Net-(U1-GND)")
+	)
+	(segment
+		(start 193.54 130.325685)
+		(end 193.305685 130.56)
+		(width 0.2)
+		(layer "F.Cu")
+		(net "Net-(U1-GND)")
+	)
+	(segment
+		(start 193.54 106.79)
+		(end 193.54 130.325685)
+		(width 0.2)
+		(layer "F.Cu")
+		(net "Net-(U1-GND)")
+	)
+	(segment
+		(start 187.945 122.445)
+		(end 187.945 107.655)
+		(width 0.2)
+		(layer "F.Cu")
+		(net "Net-(U1-GND)")
+	)
+	(segment
+		(start 186.545 102.815101)
+		(end 187.365101 101.995)
+		(width 0.2)
+		(layer "F.Cu")
+		(net "Net-(U1-GND)")
+	)
+	(segment
+		(start 157.96 130.56)
+		(end 149.845 122.445)
+		(width 0.2)
+		(layer "F.Cu")
+		(net "Net-(U1-GND)")
+	)
+	(segment
+		(start 187.945 107.655)
+		(end 186.545 106.255)
+		(width 0.2)
+		(layer "F.Cu")
+		(net "Net-(U1-GND)")
+	)
+	(segment
+		(start 193.305685 130.56)
+		(end 157.96 130.56)
+		(width 0.2)
+		(layer "F.Cu")
+		(net "Net-(U1-GND)")
+	)
+	(segment
+		(start 187.365101 101.995)
+		(end 188.745 101.995)
+		(width 0.2)
+		(layer "F.Cu")
+		(net "Net-(U1-GND)")
 	)
 	(embedded_fonts no)

Commit message: Autosave
Routing:
- net Net-(U1-PA6_A10_D10_MOSI): track 0.00 -> 130.3 mm
- net Net-(SW1-Pad2): track 0.00 -> 19.1 mm
Changed lines of the file:
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@@
+	)
+	(segment
+		(start 193.94 132.22)
+		(end 193.67 132.49)
+		(width 0.2)
+		(layer "F.Cu")
+		(net "Net-(U1-PA6_A10_D10_MOSI)")
+	)
+	(segment
+		(start 143.475 122.445)
+		(end 130.795 122.445)
+		(width 0.2)
+		(layer "F.Cu")
+		(net "Net-(U1-PA6_A10_D10_MOSI)")
+	)
+	(segment
+		(start 150.402056 123.845)
+		(end 144.875 123.845)
+		(width 0.2)
+		(layer "F.Cu")
+		(net "Net-(U1-PA6_A10_D10_MOSI)")
+	)
+	(segment
+		(start 188.910686 101.595)
+		(end 193.94 106.624315)
+		(width 0.2)
+		(layer "F.Cu")
+		(net "Net-(U1-PA6_A10_D10_MOSI)")
+	)
+	(segment
+		(start 193.94 106.624315)
+		(end 193.94 132.22)
+		(width 0.2)
+		(layer "F.Cu")
+		(net "Net-(U1-PA6_A10_D10_MOSI)")
+	)
+	(segment
+		(start 187.199416 101.595)
+		(end 188.910686 101.595)
+		(width 0.2)
+		(layer "F.Cu")
+		(net "Net-(U1-PA6_A10_D10_MOSI)")
+	)
+	(segment
+		(start 193.67 132.49)
+		(end 159.047056 132.49)
+		(width 0.2)
+		(layer "F.Cu")
+		(net "Net-(U1-PA6_A10_D10_MOSI)")
+	)
+	(segment
+		(start 168.895 121.661598)
+		(end 186.145 104.411598)
+		(width 0.2)
+		(layer "F.Cu")
+		(net "Net-(U1-PA6_A10_D10_MOSI)")
+	)
+	(segment
+		(start 159.047056 132.49)
+		(end 150.402056 123.845)
+		(width 0.2)
+		(layer "F.Cu")
+		(net "Net-(U1-PA6_A10_D10_MOSI)")
+	)
+	(segment
+		(start 168.895 122.445)
+		(end 168.895 121.661598)
+		(width 0.2)
+		(layer "F.Cu")
+		(net "Net-(U1-PA6_A10_D10_MOSI)")
+	)
+	(segment
+		(start 186.145 104.411598)
+		(end 186.145 102.649415)
+		(width 0.2)
+		(layer "F.Cu")
+		(net "Net-(U1-PA6_A10_D10_MOSI)")
+	)
+	(segment
+		(start 144.875 123.845)
+		(end 143.475 122.445)
+		(width 0.2)
+		(layer "F.Cu")
+		(net "Net-(U1-PA6_A10_D10_MOSI)")
+	)
+	(segment
+		(start 186.145 102.649415)
+		(end 187.199416 101.595)
+		(width 0.2)
+		(layer "F.Cu")
+		(net "Net-(U1-PA6_A10_D10_MOSI)")
+	)
+	(segment
+		(start 143.495 105.935)
+		(end 124.445 105.935)
+		(width 0.2)
+		(layer "F.Cu")
+		(net "Net-(SW1-Pad2)")
 	)
 	(segment

Commit message: Autosave
Routing:
- net Net-(SW1-Pad2): track 19.1 -> 57.2 mm
- net Net-(U1-PA5_A9_D9_MISO): track 0.00 -> 25.3 mm
Changed lines of the file:
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@@
+	)
+	(segment
+		(start 145.62597 88.56403)
+		(end 149.975 88.56403)
+		(width 0.2)
+		(layer "F.Cu")
+		(net "Net-(U1-PA5_A9_D9_MISO)")
+	)
+	(segment
+		(start 130.795 103.395)
+		(end 145.62597 88.56403)
+		(width 0.2)
+		(layer "F.Cu")
+		(net "Net-(U1-PA5_A9_D9_MISO)")
 	)
 	(segment
@@
 	)
 	(segment
+		(start 124.445 105.935)
+		(end 124.445 124.985)
+		(width 0.2)
+		(layer "F.Cu")
+		(net "Net-(SW1-Pad2)")
+	)
+	(segment
+		(start 124.445 124.985)
+		(end 143.495 124.985)
+		(width 0.2)
+		(layer "F.Cu")
+		(net "Net-(SW1-Pad2)")
+	)
+	(segment

Commit message: Autosave
Routing:
- net Net-(U1-PA5_A9_D9_MISO): track 25.3 -> 50.4 mm
Changed lines of the file:
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@@
+	)
+	(segment
+		(start 168.895 103.395)
+		(end 164.80597 103.395)
+		(width 0.2)
+		(layer "F.Cu")
+		(net "Net-(U1-PA5_A9_D9_MISO)")
 	)
 	(segment
@@
 		(width 0.2)
 		(layer "F.Cu")
+		(net "Net-(U1-PA5_A9_D9_MISO)")
+	)
+	(segment
+		(start 164.80597 103.395)
+		(end 149.975 88.56403)
+		(width 0.2)
+		(layer "F.Cu")
