File: PCB/TheGitboard2.0/TheGitboard2.0.kicad_pcb (KiCad board)
At the start: 2 copper layers, 78.3 x 70.1 mm, 9 parts, among them SW1 SW_Push, SW2 SW_Push, SW3 SW_Push, SW4 SW_Push, SW5 SW_Push, SW6 SW_Push, SW7 SW_Push, SW8 SW_Push, U1 MOUDLE-SEEEDUINO-XIAO

Commit message: Aug 13, 2026, 5:17 PM
Parts:
- moved U1 6.69 mm to (157.6, 86.0)
- moved SW1 3.76 mm to (130.8, 105.5)
- moved SW2 3.76 mm to (130.8, 124.5)
- moved SW3 3.76 mm to (149.8, 105.5)
- moved SW4 3.76 mm to (149.8, 124.5)
- moved SW5 3.76 mm to (168.9, 105.5)
- moved SW6 3.76 mm to (168.9, 124.5)
- moved SW7 3.76 mm to (187.9, 105.5)
- moved SW8 3.76 mm to (187.9, 124.5)
Routing:
- net Net-(U1-PA6_A10_D10_MOSI): track 115.5 -> 146.5 mm
- net Net-(U1-GND): track 125.6 -> 152.3 mm
- net Net-(U1-3V3): track 85.3 -> 92.1 mm
- net Net-(U1-PA7_A8_D8_SCK): track 85.6 -> 91.3 mm
- net Net-(U1-PA5_A9_D9_MISO): track 56.8 -> 52.1 mm
